File: ExternalAutoprogramming.kicad_sch (KiCad schematic)
At the start: 1 part, among them J4 Conn_01x04_Socket

Commit message: feat: Remove BOOT pin connection
Connections:
- net BOOT: no longer names the net of J4.4 (BOOT)
- no-connect marks 0 -> 1
Changed lines of the file:
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@@
 		(company "Vynte")
+	)
+	(no_connect
+		(at 168.91 96.52)
 	)
 	(wire
@@
 		(effects
 			(font
-				(size 1.27 1.27)
-			)
-			(justify left)
-		)
-	)
-	(hierarchical_label "BOOT"
-		(shape bidirectional)
-		(at 168.91 96.52 0)
-		(effects
-			(font

Commit message: feat: Disconnected the VCC pin from external autoprogramming
Connections:
- net +3.3V: no longer names the net of J4.5 (VCC)
- no-connect marks 1 -> 2
Changed lines of the file:
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@@
 		(at 168.91 96.52)
 	)
-	(wire
-		(pts
-			(xy 139.7 99.06) (xy 149.86 99.06)
-		)
-		(stroke
-			(width 0)
-			(type default)
-		)
+	(no_connect
+		(at 149.86 99.06)
 	)
 	(wire
 		(pts
 			(xy 171.45 99.06) (xy 168.91 99.06)
-		)
-		(stroke
-			(width 0)
-			(type default)
-		)
-	)
-	(wire
-		(pts
-			(xy 139.7 96.52) (xy 139.7 99.06)
 		)
 		(stroke
@@
 					(unit 1)
 				)
-			)
-		)
-	)
-	(symbol
-		(lib_id "power:+3.3V")
-		(at 139.7 96.52 0)
-		(unit 1)
-		(body_style 1)
-		(exclude_from_sim no)
-		(in_bom yes)
-		(on_board yes)
-		(in_pos_files yes)
-		(dnp no)
-		(fields_autoplaced yes)
-		(property "Reference" "#PWR06"
-			(at 139.7 100.33 0)
-			(hide yes)
-			(show_name no)
-			(do_not_autoplace no)
-			(effects
-				(font
-					(size 1.27 1.27)
-				)
-			)
-		)
-		(property "Value" "+3.3V"
-			(at 139.7 91.44 0)
-			(show_name no)
-			(do_not_autoplace no)
-			(effects
-				(font
-					(size 1.27 1.27)
-				)
-			)
-		)
-		(property "Footprint" ""
-			(at 139.7 96.52 0)
-			(hide yes)
-			(show_name no)
-			(do_not_autoplace no)
-			(effects
-				(font
-					(size 1.27 1.27)
-				)
-			)
-		)
-		(property "Datasheet" ""
-			(at 139.7 96.52 0)
-			(hide yes)
-			(show_name no)
-			(do_not_autoplace no)
-			(effects
-				(font
-					(size 1.27 1.27)
-				)
-			)
-		)
-		(property "Description" "Power symbol creates a global label with name \"+3.3V\""
-			(at 139.7 96.52 0)
-			(hide yes)
-			(show_name no)
-			(do_not_autoplace no)
-			(effects
-				(font
-					(size 1.27 1.27)
-				)
-			)
-		)
-		(pin "1"
-		)
-		(instances
-			(project "Vent"
-				(path "/44080430-3c3a-4a58-87da-65c26034d41d/baa2a2d6-ded2-444d-b992-886e8249722c"
-					(reference "#PWR06")
-					(unit 1)
-				)
