File: ExternalAutoprogramming.kicad_sch (KiCad schematic)
At the start: 1 part, among them J4 Conn_01x04_Socket

Commit message: feat: Add metadata and version to sheets
Other:
- title: (none) -> Vent
Changed lines of the file:
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@@
 	(generator_version "10.0")
 	(paper "A4")
+	(title_block
+		(title "Vent")
+		(date "2026-08-19")
+		(rev "v0.1.0")
+	)
 	(wire
 		(pts
@@
 		)
 		(instances
-			(project "Vynte PCB"
+			(project "Vent"
 				(path "/44080430-3c3a-4a58-87da-65c26034d41d/baa2a2d6-ded2-444d-b992-886e8249722c"
 					(reference "J4")
@@
 		)
 		(instances
-			(project "Vynte PCB"
+			(project "Vent"
 				(path "/44080430-3c3a-4a58-87da-65c26034d41d/baa2a2d6-ded2-444d-b992-886e8249722c"
 					(reference "#PWR06")
@@
 		)
 		(instances
-			(project "Vynte PCB"
+			(project "Vent"
 				(path "/44080430-3c3a-4a58-87da-65c26034d41d/baa2a2d6-ded2-444d-b992-886e8249722c"
 					(reference "#PWR05")

Commit message: Schematic Organization
Connections:
- net D+ renamed RX
- net D- renamed TX
Changed lines of the file:
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@@
 		)
 	)
-	(hierarchical_label "D-"
+	(hierarchical_label "TX"
 		(shape bidirectional)
 		(at 149.86 96.52 180)
@@
 		)
 	)
-	(hierarchical_label "D+"
+	(hierarchical_label "RX"
 		(shape bidirectional)
 		(at 149.86 93.98 180)

Commit message: fix: Fix individual sheet names
Other:
- title: Vent -> External Autoprogramming
Changed lines of the file:
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@@
 	(paper "A4")
 	(title_block
-		(title "Vent")
+		(title "External Autoprogramming")
 		(date "2026-08-19")
 		(rev "${PROJECT_REV}")

Commit message: fix: Add company name to schematic sheets
Other:
- company: (none) -> Vynte
Changed lines of the file:
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@@
 		(date "2026-08-19")
 		(rev "${PROJECT_REV}")
+		(company "Vynte")
 	)
 	(wire

Commit message: replace tx0 and rx0 with D+ and D-
Connections:
- net RX renamed D-
- net TX renamed D+
Changed lines of the file:
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@@
 		)
 	)
-	(hierarchical_label "TX"
+	(hierarchical_label "D+"
 		(shape bidirectional)
 		(at 149.86 96.52 180)
@@
 		)
 	)
-	(hierarchical_label "RX"
+	(hierarchical_label "D-"
 		(shape bidirectional)
 		(at 149.86 93.98 180)

Commit message: metadata
Parts:
- J4: MPN (none) -> TC2030-IDC-NL; Manufacturer (none) -> Tag-Connect
Changed lines of the file:
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@@
+			)
+		)
+		(property "Manufacturer" "Tag-Connect" (at 0 0 0)
+			(effects
+				(font
+					(size 1.27 1.27)
+				)
+				(hide yes)
+			)
+		)
+		(property "MPN" "TC2030-IDC-NL" (at 0 0 0)
+			(effects
+				(font
+					(size 1.27 1.27)
+				)
+				(hide yes)
 			)
 		)
