File: 3.3V-Buck-Boost.kicad_sch (KiCad schematic)
At the start: 6 parts, among them U4 MCP1640x-xMC

Commit message: feat: Add metadata and version to sheets
Other:
- title: (none) -> Vent
Changed lines of the file:
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@@
 	(generator_version "10.0")
 	(paper "A4")
+	(title_block
+		(title "Vent")
+		(date "2026-08-19")
+		(rev "v0.1.0")
+	)
 	(junction
 		(at 135.89 102.87)
@@
 		)
 		(instances
-			(project "Vynte PCB"
+			(project "Vent"
 				(path "/44080430-3c3a-4a58-87da-65c26034d41d/cbe65d49-7ad3-41aa-a0de-e365567d2c38"
 					(reference "#PWR025")
@@
 		)
 		(instances
-			(project "Vynte PCB"
+			(project "Vent"
 				(path "/44080430-3c3a-4a58-87da-65c26034d41d/cbe65d49-7ad3-41aa-a0de-e365567d2c38"
 					(reference "#PWR027")
@@
 		)
 		(instances
-			(project "Vynte PCB"
+			(project "Vent"
 				(path "/44080430-3c3a-4a58-87da-65c26034d41d/cbe65d49-7ad3-41aa-a0de-e365567d2c38"
 					(reference "#PWR026")
@@
 		)
 		(instances
-			(project "Vynte PCB"
+			(project "Vent"
 				(path "/44080430-3c3a-4a58-87da-65c26034d41d/cbe65d49-7ad3-41aa-a0de-e365567d2c38"
 					(reference "U4")
@@
 		)
 		(instances
-			(project "Vynte PCB"
+			(project "Vent"
 				(path "/44080430-3c3a-4a58-87da-65c26034d41d/cbe65d49-7ad3-41aa-a0de-e365567d2c38"
 					(reference "C_{OUT}2")
@@
 		)
 		(instances
-			(project "Vynte PCB"
+			(project "Vent"
 				(path "/44080430-3c3a-4a58-87da-65c26034d41d/cbe65d49-7ad3-41aa-a0de-e365567d2c38"
 					(reference "C_{IN}2")
@@
 		)
 		(instances
-			(project "Vynte PCB"
+			(project "Vent"
 				(path "/44080430-3c3a-4a58-87da-65c26034d41d/cbe65d49-7ad3-41aa-a0de-e365567d2c38"
 					(reference "#PWR023")
@@
 		)
 		(instances
-			(project "Vynte PCB"
+			(project "Vent"
 				(path "/44080430-3c3a-4a58-87da-65c26034d41d/cbe65d49-7ad3-41aa-a0de-e365567d2c38"
 					(reference "#PWR024")
@@
 		)
 		(instances
-			(project "Vynte PCB"
+			(project "Vent"
 				(path "/44080430-3c3a-4a58-87da-65c26034d41d/cbe65d49-7ad3-41aa-a0de-e365567d2c38"
 					(reference "R_{BOT}2")
@@
 		)
 		(instances
-			(project "Vynte PCB"
+			(project "Vent"
 				(path "/44080430-3c3a-4a58-87da-65c26034d41d/cbe65d49-7ad3-41aa-a0de-e365567d2c38"
 					(reference "L3")
@@
 		)
 		(instances
-			(project "Vynte PCB"
+			(project "Vent"
 				(path "/44080430-3c3a-4a58-87da-65c26034d41d/cbe65d49-7ad3-41aa-a0de-e365567d2c38"
 					(reference "R_{TOP}2")

Commit message: fix: Fix individual sheet names
Other:
- title: Vent -> 3.3V Buck-Boost Voltage Regulator
Changed lines of the file:
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@@
 	(paper "A4")
 	(title_block
-		(title "Vent")
+		(title "3.3V Buck-Boost Voltage Regulator")
 		(date "2026-08-19")
 		(rev "${PROJECT_REV}")

Commit message: fix: Add company name to schematic sheets
Other:
- company: (none) -> Vynte
Changed lines of the file:
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@@
 		(date "2026-08-19")
 		(rev "${PROJECT_REV}")
+		(company "Vynte")
 	)
 	(junction

Commit message: metadata
Parts:
- C_{IN}2: Digi-Key_PN (none) -> 587-2990-1-ND; MPN (none) -> TMK212AB7475KG-T; Manufacturer (none) -> Taiyo Yuden
- C_{OUT}2: Digi-Key_PN (none) -> 587-4334-1-ND; MPN (none) -> TMK212BBJ106KGHT; Manufacturer (none) -> Taiyo Yuden
- L3: Digi-Key_PN (none) -> 240-TYA30124R7M-10CT-ND; MPN (none) -> TYA30124R7M-10; Manufacturer (none) -> Laird-Signal Integrity Products
- R_{BOT}2: Digi-Key_PN (none) -> 311-309KHRCT-ND; MPN (none) -> RC0603FR-07309KL; Manufacturer (none) -> YAGEO
- R_{TOP}2: Digi-Key_PN (none) -> 311-536KHRCT-ND; MPN (none) -> RC0603FR-07536KL; Manufacturer (none) -> YAGEO
- U4: Digi-Key_PN (none) -> MCP1640CT-I/MCCT-ND; MPN (none) -> MCP1640CT-I/MC; Manufacturer (none) -> Microchip Technology
Changed lines of the file:
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@@
+			)
+		)
+		(property "Digi-Key_PN" "MCP1640CT-I/MCCT-ND" (at 0 0 0)
+			(effects
+				(font
+					(size 1.27 1.27)
+				)
+				(hide yes)
+			)
+		)
+		(property "Manufacturer" "Microchip Technology" (at 0 0 0)
+			(effects
+				(font
+					(size 1.27 1.27)
+				)
+				(hide yes)
+			)
+		)
+		(property "MPN" "MCP1640CT-I/MC" (at 0 0 0)
+			(effects
+				(font
+					(size 1.27 1.27)
+				)
+				(hide yes)
 			)
 		)
@@
 			)
 		)
+		(property "Digi-Key_PN" "587-4334-1-ND" (at 0 0 0)
+			(effects
+				(font
+					(size 1.27 1.27)
+				)
+				(hide yes)
+			)
+		)
+		(property "Manufacturer" "Taiyo Yuden" (at 0 0 0)
+			(effects
+				(font
+					(size 1.27 1.27)
+				)
+				(hide yes)
+			)
+		)
+		(property "MPN" "TMK212BBJ106KGHT" (at 0 0 0)
+			(effects
+				(font
+					(size 1.27 1.27)
+				)
+				(hide yes)
+			)
+		)
 		(pin "1"
 		)
@@
 			)
 		)
+		(property "Digi-Key_PN" "587-2990-1-ND" (at 0 0 0)
+			(effects
+				(font
+					(size 1.27 1.27)
+				)
+				(hide yes)
+			)
+		)
+		(property "Manufacturer" "Taiyo Yuden" (at 0 0 0)
+			(effects
+				(font
+					(size 1.27 1.27)
+				)
+				(hide yes)
+			)
+		)
+		(property "MPN" "TMK212AB7475KG-T" (at 0 0 0)
+			(effects
+				(font
+					(size 1.27 1.27)
+				)
+				(hide yes)
+			)
+		)
 		(pin "2"
 		)
@@
 			)
 		)
+		(property "Digi-Key_PN" "311-309KHRCT-ND" (at 0 0 0)
+			(effects
+				(font
+					(size 1.27 1.27)
+				)
+				(hide yes)
+			)
+		)
+		(property "Manufacturer" "YAGEO" (at 0 0 0)
+			(effects
+				(font
+					(size 1.27 1.27)
+				)
+				(hide yes)
+			)
+		)
+		(property "MPN" "RC0603FR-07309KL" (at 0 0 0)
+			(effects
+				(font
+					(size 1.27 1.27)
+				)
+				(hide yes)
+			)
+		)
 		(pin "1"
 		)
@@
 					(size 1.27 1.27)
 				)
+			)
+		)
+		(property "Digi-Key_PN" "240-TYA30124R7M-10CT-ND" (at 0 0 0)
+			(effects
+				(font
+					(size 1.27 1.27)
+				)
+				(hide yes)
+			)
+		)
+		(property "Manufacturer" "Laird-Signal Integrity Products" (at 0 0 0)
+			(effects
+				(font
+					(size 1.27 1.27)
+				)
+				(hide yes)
+			)
+		)
+		(property "MPN" "TYA30124R7M-10" (at 0 0 0)
+			(effects
+				(font
+					(size 1.27 1.27)
+				)
+				(hide yes)
 			)
 		)
@@
 			)
 		)
+		(property "Digi-Key_PN" "311-536KHRCT-ND" (at 0 0 0)
+			(effects
+				(font
+					(size 1.27 1.27)
+				)
+				(hide yes)
+			)
+		)
+		(property "Manufacturer" "YAGEO" (at 0 0 0)
+			(effects
+				(font
+					(size 1.27 1.27)
+				)
+				(hide yes)
+			)
+		)
+		(property "MPN" "RC0603FR-07536KL" (at 0 0 0)
+			(effects
+				(font
+					(size 1.27 1.27)
+				)
+				(hide yes)
+			)
+		)
