File: 5V-Boost.kicad_sch (KiCad schematic)
At the start: 8 parts

Commit message: feat: Add metadata and version to sheets
Other:
- title: (none) -> Vent
Changed lines of the file:
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@@
 	(generator_version "10.0")
 	(paper "A4")
+	(title_block
+		(title "Vent")
+		(date "2026-08-19")
+		(rev "v0.1.0")
+	)
 	(junction
 		(at 173.99 85.09)
@@
 		)
 		(instances
-			(project "Vynte PCB"
+			(project "Vent"
 				(path "/44080430-3c3a-4a58-87da-65c26034d41d/2412c928-f5bc-4770-b369-2941957c7d2e"
 					(reference "#PWR010")
@@
 		)
 		(instances
-			(project "Vynte PCB"
+			(project "Vent"
 				(path "/44080430-3c3a-4a58-87da-65c26034d41d/2412c928-f5bc-4770-b369-2941957c7d2e"
 					(reference "R3")
@@
 		)
 		(instances
-			(project "Vynte PCB"
+			(project "Vent"
 				(path "/44080430-3c3a-4a58-87da-65c26034d41d/2412c928-f5bc-4770-b369-2941957c7d2e"
 					(reference "C1")
@@
 		)
 		(instances
-			(project "Vynte PCB"
+			(project "Vent"
 				(path "/44080430-3c3a-4a58-87da-65c26034d41d/2412c928-f5bc-4770-b369-2941957c7d2e"
 					(reference "#PWR09")
@@
 		)
 		(instances
-			(project "Vynte PCB"
+			(project "Vent"
 				(path "/44080430-3c3a-4a58-87da-65c26034d41d/2412c928-f5bc-4770-b369-2941957c7d2e"
 					(reference "R2")
@@
 		)
 		(instances
-			(project "Vynte PCB"
+			(project "Vent"
 				(path "/44080430-3c3a-4a58-87da-65c26034d41d/2412c928-f5bc-4770-b369-2941957c7d2e"
 					(reference "C3")
@@
 		)
 		(instances
-			(project "Vynte PCB"
+			(project "Vent"
 				(path "/44080430-3c3a-4a58-87da-65c26034d41d/2412c928-f5bc-4770-b369-2941957c7d2e"
 					(reference "C2")
@@
 		)
 		(instances
-			(project "Vynte PCB"
+			(project "Vent"
 				(path "/44080430-3c3a-4a58-87da-65c26034d41d/2412c928-f5bc-4770-b369-2941957c7d2e"
 					(reference "L1")
@@
 		)
 		(instances
-			(project "Vynte PCB"
+			(project "Vent"
 				(path "/44080430-3c3a-4a58-87da-65c26034d41d/2412c928-f5bc-4770-b369-2941957c7d2e"
 					(reference "R1")
@@
 		)
 		(instances
-			(project "Vynte PCB"
+			(project "Vent"
 				(path "/44080430-3c3a-4a58-87da-65c26034d41d/2412c928-f5bc-4770-b369-2941957c7d2e"
 					(reference "#PWR08")
@@
 		)
 		(instances
-			(project "Vynte PCB"
+			(project "Vent"
 				(path "/44080430-3c3a-4a58-87da-65c26034d41d/2412c928-f5bc-4770-b369-2941957c7d2e"
 					(reference "#PWR03")
@@
 		)
 		(instances
-			(project "Vynte PCB"
+			(project "Vent"
 				(path "/44080430-3c3a-4a58-87da-65c26034d41d/2412c928-f5bc-4770-b369-2941957c7d2e"
 					(reference "#PWR07")
@@
 		)
 		(instances
-			(project "Vynte PCB"
+			(project "Vent"
 				(path "/44080430-3c3a-4a58-87da-65c26034d41d/2412c928-f5bc-4770-b369-2941957c7d2e"
 					(reference "U2")

Commit message: fix: Fix individual sheet names
Other:
- title: Vent -> 5V Boost Voltage Regulator
Changed lines of the file:
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@@
 	(paper "A4")
 	(title_block
-		(title "Vent")
+		(title "5V Boost Voltage Regulator")
 		(date "2026-08-19")
 		(rev "${PROJECT_REV}")

Commit message: fix: Add company name to schematic sheets
Other:
- company: (none) -> Vynte
Changed lines of the file:
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@@
 		(date "2026-08-19")
 		(rev "${PROJECT_REV}")
+		(company "Vynte")
 	)
 	(junction

Commit message: metadata
Parts:
- C1, C2, C3: Digi-Key_PN (none) -> 587-3246-1-ND; MPN (none) -> TMK316BBJ226ML-T; Manufacturer (none) -> Taiyo Yuden
- L1: Digi-Key_PN (none) -> 732-11197-1-ND; MPN (none) -> 74438357010; Manufacturer (none) -> Würth Elektronik
- R1: Digi-Key_PN (none) -> P732KHCT-ND; MPN (none) -> ERJ-3EKF7323V; Manufacturer (none) -> Panasonic Industry
- R2, R3: Digi-Key_PN (none) -> 311-100KHRCT-ND; MPN (none) -> RC0603FR-07100KL; Manufacturer (none) -> YAGEO
- U2: Digi-Key_PN (none) -> 296-TPS61023DRLRCT-ND; MPN (none) -> TPS61023DRLR; Manufacturer (none) -> Texas Instruments
Changed lines of the file:
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@@
+			)
+		)
+		(property "Digi-Key_PN" "311-100KHRCT-ND" (at 0 0 0)
+			(effects
+				(font
+					(size 1.27 1.27)
+				)
+				(hide yes)
+			)
+		)
+		(property "Manufacturer" "YAGEO" (at 0 0 0)
+			(effects
+				(font
+					(size 1.27 1.27)
+				)
+				(hide yes)
+			)
+		)
+		(property "MPN" "RC0603FR-07100KL" (at 0 0 0)
+			(effects
+				(font
+					(size 1.27 1.27)
+				)
+				(hide yes)
 			)
 		)
@@
 					(size 1.27 1.27)
 				)
+			)
+		)
+		(property "Digi-Key_PN" "587-3246-1-ND" (at 0 0 0)
+			(effects
+				(font
+					(size 1.27 1.27)
+				)
+				(hide yes)
+			)
+		)
+		(property "Manufacturer" "Taiyo Yuden" (at 0 0 0)
+			(effects
+				(font
+					(size 1.27 1.27)
+				)
+				(hide yes)
+			)
+		)
+		(property "MPN" "TMK316BBJ226ML-T" (at 0 0 0)
+			(effects
+				(font
+					(size 1.27 1.27)
+				)
+				(hide yes)
 			)
 		)
@@
 			)
 		)
+		(property "Digi-Key_PN" "311-100KHRCT-ND" (at 0 0 0)
+			(effects
+				(font
+					(size 1.27 1.27)
+				)
+				(hide yes)
+			)
+		)
+		(property "Manufacturer" "YAGEO" (at 0 0 0)
+			(effects
+				(font
+					(size 1.27 1.27)
+				)
+				(hide yes)
+			)
+		)
+		(property "MPN" "RC0603FR-07100KL" (at 0 0 0)
+			(effects
+				(font
+					(size 1.27 1.27)
+				)
+				(hide yes)
+			)
+		)
 		(pin "1"
 		)
@@
 			)
 		)
+		(property "Digi-Key_PN" "587-3246-1-ND" (at 0 0 0)
+			(effects
+				(font
+					(size 1.27 1.27)
+				)
+				(hide yes)
+			)
+		)
+		(property "Manufacturer" "Taiyo Yuden" (at 0 0 0)
+			(effects
+				(font
+					(size 1.27 1.27)
+				)
+				(hide yes)
+			)
+		)
+		(property "MPN" "TMK316BBJ226ML-T" (at 0 0 0)
+			(effects
+				(font
+					(size 1.27 1.27)
+				)
+				(hide yes)
+			)
+		)
 		(pin "1"
 		)
@@
 					(size 1.27 1.27)
 				)
+			)
+		)
+		(property "Digi-Key_PN" "587-3246-1-ND" (at 0 0 0)
+			(effects
+				(font
+					(size 1.27 1.27)
+				)
+				(hide yes)
+			)
+		)
+		(property "Manufacturer" "Taiyo Yuden" (at 0 0 0)
+			(effects
+				(font
+					(size 1.27 1.27)
+				)
+				(hide yes)
+			)
+		)
+		(property "MPN" "TMK316BBJ226ML-T" (at 0 0 0)
+			(effects
+				(font
+					(size 1.27 1.27)
+				)
+				(hide yes)
 			)
 		)
@@
 			)
 		)
+		(property "Digi-Key_PN" "732-11197-1-ND" (at 0 0 0)
+			(effects
+				(font
+					(size 1.27 1.27)
+				)
+				(hide yes)
+			)
+		)
+		(property "Manufacturer" "Würth Elektronik" (at 0 0 0)
+			(effects
+				(font
+					(size 1.27 1.27)
+				)
+				(hide yes)
+			)
+		)
+		(property "MPN" "74438357010" (at 0 0 0)
+			(effects
+				(font
+					(size 1.27 1.27)
+				)
+				(hide yes)
+			)
+		)
 		(pin "2"
 		)
@@
 			)
 		)
+		(property "Digi-Key_PN" "P732KHCT-ND" (at 0 0 0)
+			(effects
+				(font
+					(size 1.27 1.27)
+				)
+				(hide yes)
+			)
+		)
+		(property "Manufacturer" "Panasonic Industry" (at 0 0 0)
+			(effects
+				(font
+					(size 1.27 1.27)
+				)
+				(hide yes)
+			)
+		)
+		(property "MPN" "ERJ-3EKF7323V" (at 0 0 0)
+			(effects
+				(font
+					(size 1.27 1.27)
+				)
+				(hide yes)
+			)
+		)
 		(pin "1"
 		)
@@
 			)
 		)
+		(property "Digi-Key_PN" "296-TPS61023DRLRCT-ND" (at 0 0 0)
+			(effects
+				(font
+					(size 1.27 1.27)
+				)
+				(hide yes)
+			)
+		)
+		(property "Manufacturer" "Texas Instruments" (at 0 0 0)
+			(effects
+				(font
+					(size 1.27 1.27)
+				)
+				(hide yes)
+			)
+		)
+		(property "MPN" "TPS61023DRLR" (at 0 0 0)
+			(effects
+				(font
+					(size 1.27 1.27)
+				)
+				(hide yes)
+			)
+		)
