File: 5V-Boost.kicad_sch (KiCad schematic)
At the start: 8 parts

Commit message: feat: Sync saved vent v0.5.0 design and fabrication package
Parts:
- C1, C2, C3: Digi-Key_PN (none) -> 1276-3047-2-ND; MPN (none) -> CL31A226KAHNNNE; Manufacturer (none) -> Samsung Electro-Mechanics
- L1: footprint Inductor_SMD:L_Wuerth_MAPI-4030 -> Inductor_SMD:L_Murata_DFE201610P; Digi-Key_PN (none) -> 490-16593-2-ND; MPN (none) -> DFE201612E-1R0M=P2; Manufacturer (none) -> Murata Electronics
- R1: Digi-Key_PN (none) -> 311-732KHRTR-ND; MPN (none) -> RC0603FR-07732KL; Manufacturer (none) -> YAGEO
- R2, R3: Digi-Key_PN (none) -> 311-100KHRTR-ND; MPN (none) -> RC0603FR-07100KL; Manufacturer (none) -> YAGEO
- U2: Digi-Key_PN (none) -> 296-TPS61023DRLRTR-ND; MPN (none) -> TPS61023DRLR; Manufacturer (none) -> Texas Instruments
