File: Vent.kicad_sch (KiCad schematic)
At the start: 11 parts, among them J2 B2B-XH-A_LF__SN_, J3 Conn_01x03_Pin, SW1 SW_Push, U1 ESP32-H2-MINI-1

Commit message: feat: Sync saved vent v0.5.0 design and fabrication package
Parts:
- removed H4: MountingHole, MountingHole:MountingHole_2.2mm_M2, symbol Mechanical:MountingHole
- C5: footprint Capacitor_SMD:C_0201_0603Metric -> Capacitor_SMD:C_0402_1005Metric; Digi-Key_PN (none) -> 445-7348-2-ND; MPN (none) -> C1005X7R1E104K050BB; Manufacturer (none) -> TDK
- D1: Digi-Key_PN (none) -> 754-1603-ND; MPN (none) -> WP710A10GD; Manufacturer (none) -> Kingbright
- J2: BOM Comments (none) -> Wire-solder pads (SolderWire footprint) - no board connecto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
- J3: BOM Comments (none) -> Wire-solder pads - 3 wires soldered directly. No connector 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
- R5: footprint Resistor_SMD:R_0201_0603Metric -> Resistor_SMD:R_0402_1005Metric; Digi-Key_PN (none) -> 311-1.00MLRTR-ND; MPN (none) -> RC0402FR-071ML; Manufacturer (none) -> YAGEO
- R6: footprint Resistor_SMD:R_0201_0603Metric -> Resistor_SMD:R_0402_1005Metric; Digi-Key_PN (none) -> 311-330KLRTR-ND; MPN (none) -> RC0402FR-07330KL; Manufacturer (none) -> YAGEO
- R7: footprint Resistor_SMD:R_0201_0603Metric -> Resistor_SMD:R_0402_1005Metric; Digi-Key_PN (none) -> 311-220LRTR-ND; MPN (none) -> RC0402FR-07220RL; Manufacturer (none) -> YAGEO
- SW1: footprint Button_Switch_SMD:SW_SPST_PTS810 -> Button_Switch_THT:SW_PUSH_6mm_H5mm; Digi-Key_PN (none) -> CKN10503TR-ND; MPN (none) -> PTS810SJK250SMTR LFS; Manufacturer (none) -> C&K
- U1: Digi-Key_PN (none) -> 1965-ESP32-H2-MINI-1-H2STR-ND; MPN (none) -> ESP32-H2-MINI-1-H2S; Manufacturer (none) -> Espressif Systems
